Commit message: bcr arm pick and place demo sim

File: src/bcr_arm_description/urdf/bcr_arm.urdf.xacro (robot description, xacro)
@@ -5,4 +5,5 @@
 <xacro:include filename="$(find bcr_arm_description)/urdf/bcr_arm_materials.xacro"/>
 <xacro:include filename="$(find bcr_arm_description)/urdf/bcr_arm_links_macros.xacro"/>
+<xacro:include filename="$(find bcr_arm_description)/urdf/gripper.xacro"/>
   <!-- ========================= -->
   <!-- Fixed world frame for Gazebo -->
@@ -84,5 +85,5 @@
     <origin xyz="0 0 0.35" rpy="0 0 0"/>
     <axis xyz="0 1 0"/>
-    <limit lower="-2.2" upper="2.2" effort="100.0" velocity="1.5"/>
+    <limit lower="-3.1416" upper="3.1416" effort="100.0" velocity="1.5"/>
   </joint>
   <!-- joint4: wrist roll -->
@@ -100,5 +101,5 @@
     <origin xyz="0 0 0.25" rpy="0 0 0"/>
     <axis xyz="0 1 0"/>
-    <limit lower="-2.2" upper="2.2" effort="80.0" velocity="1.5"/>
+    <limit lower="-3.1416" upper="3.1416" effort="80.0" velocity="1.5"/>
   </joint>
   <!-- joint6: wrist roll -->
@@ -116,5 +117,5 @@
     <origin xyz="0 0 0.16" rpy="0 0 0"/>
     <axis xyz="0 1 0"/>
-    <limit lower="-2.2" upper="2.2" effort="60.0" velocity="1.5"/>
+    <limit lower="-3.1416" upper="3.1416" effort="60.0" velocity="1.5"/>
   </joint>
   <!-- fixed tool joint -->
@@ -124,4 +125,5 @@
     <origin xyz="0 0 0.12" rpy="0 0 0"/>
   </joint>
+  <xacro:bcr_arm_fixed_gripper parent_link="tool0" prefix="gripper_"/>
 <!-- ros2_control 硬件接口 + Gazebo 插件 -->
 <!-- 加载控制器配置文件，连接仿真器与控制系统 -->

File: src/bcr_arm_description/urdf/bcr_arm_ros2_controllers.xacro (robot description, xacro)
@@ -46,6 +46,16 @@
         <state_interface name="velocity"/>
       </joint>
+       <!-- gripper joints -->
+      <joint name="gripper_left_finger_joint">
+        <command_interface name="position"/>
+        <state_interface name="position"/>
+        <state_interface name="velocity"/>
+      </joint>
+      <joint name="gripper_right_finger_joint">
+        <command_interface name="position"/>
+        <state_interface name="position"/>
+        <state_interface name="velocity"/>
+      </joint>
     </ros2_control>
-    <!-- Gazebo 插件，加载控制器 YAML 配置 -->
     <gazebo>
       <plugin filename="ign_ros2_control-system"

File: src/bcr_arm_moveit_config/config/bcr_arm.urdf.xacro (robot description, xacro)
@@ -3,5 +3,5 @@
     <xacro:arg name="initial_positions_file" default="initial_positions.yaml" />
     <!-- Import bcr_arm urdf file -->
-    <xacro:include filename="$(find bcr_arm_description)/urdf/bcr_arm.urdf" />
+    <xacro:include filename="$(find bcr_arm_description)/urdf/bcr_arm.urdf.xacro" />
     <!-- Import control_xacro -->
     <xacro:include filename="bcr_arm.ros2_control.xacro" />
